File: clickclack-mk-1.1-a.sch (EAGLE design)
At the start: 20 parts, among them SW1 CHERRY-MXNONUBS, SW2 CHERRY-MXNONUBS, SW3 CHERRY-MXNONUBS, SW4 CHERRY-MXNONUBS, SW5 CHERRY-MXNONUBS, SW6 CHERRY-MXNONUBS, U1 TEENSY_3.0_BASIC_ALTDIP

Commit message: [wip] do not use
Parts:
- removed C1, C2: 100n, A_butts:CAPACITOR-CERAMIC025-024X044
- removed D4, D5, D6: 1N4148, A_butts:DIODEPTH-7.62MM
- removed SW4, SW5, SW6: CHERRY-MXNONUBS, A_butts:CHERRY-MXNONUBS
Connections:
- removed net N$4: D4.A, SW4.COM
- removed net N$5: D5.A, SW5.COM
- removed net N$6: D6.A, SW6.COM
- net GND: no longer C1.2, C2.2, D4.C, D5.C, D6.C
- net KEY4: no longer SW4.NO
- net KEY5: no longer SW5.NO
- net KEY6: no longer SW6.NO
- net VCC: no longer C1.1, C2.1
Changed lines of the file:
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@@
 <part name="SW2" library="A_butts" deviceset="CHERRY-MX" device="NONUBS" value="CHERRY-MXNONUBS"/>
 <part name="SW3" library="A_butts" deviceset="CHERRY-MX" device="NONUBS" value="CHERRY-MXNONUBS"/>
-<part name="SW4" library="A_butts" deviceset="CHERRY-MX" device="NONUBS" value="CHERRY-MXNONUBS"/>
-<part name="SW5" library="A_butts" deviceset="CHERRY-MX" device="NONUBS" value="CHERRY-MXNONUBS"/>
-<part name="SW6" library="A_butts" deviceset="CHERRY-MX" device="NONUBS" value="CHERRY-MXNONUBS"/>
 <part name="D1" library="A_butts" deviceset="DIODE" device="PTH-7.62MM" value="1N4148"/>
 <part name="D2" library="A_butts" deviceset="DIODE" device="PTH-7.62MM" value="1N4148"/>
 <part name="D3" library="A_butts" deviceset="DIODE" device="PTH-7.62MM" value="1N4148"/>
-<part name="D4" library="A_butts" deviceset="DIODE" device="PTH-7.62MM" value="1N4148"/>
-<part name="D5" library="A_butts" deviceset="DIODE" device="PTH-7.62MM" value="1N4148"/>
-<part name="D6" library="A_butts" deviceset="DIODE" device="PTH-7.62MM" value="1N4148"/>
 <part name="SUPPLY2" library="A_butts" deviceset="VCC" device=""/>
 <part name="GND2" library="A_butts" deviceset="GND" device=""/>
@@
 <part name="U1" library="A_butts" deviceset="TEENSY_3.0_BASIC_ALT" device="DIP"/>
 <part name="GND4" library="A_butts" deviceset="GND" device=""/>
-<part name="SUPPLY1" library="A_butts" deviceset="VCC" device=""/>
-<part name="C1" library="A_butts" deviceset="CAPACITOR-CERAMIC" device="025-024X044" value="100n"/>
-<part name="C2" library="A_butts" deviceset="CAPACITOR-CERAMIC" device="025-024X044" value="100n"/>
-<part name="SUPPLY4" library="A_butts" deviceset="VCC" device=""/>
-<part name="GND1" library="A_butts" deviceset="GND" device=""/>
-<part name="GND5" library="A_butts" deviceset="GND" device=""/>
 </parts>
 <sheets>
@@
 <instance part="SW2" gate="G$1" x="50.8" y="144.78" rot="MR0"/>
 <instance part="SW3" gate="G$1" x="50.8" y="137.16" rot="MR0"/>
-<instance part="SW4" gate="G$1" x="50.8" y="129.54" rot="MR0"/>
-<instance part="SW5" gate="G$1" x="50.8" y="121.92" rot="MR0"/>
-<instance part="SW6" gate="G$1" x="50.8" y="114.3" rot="MR0"/>
 <instance part="D1" gate="G$1" x="60.96" y="152.4"/>
 <instance part="D2" gate="G$1" x="60.96" y="144.78"/>
 <instance part="D3" gate="G$1" x="60.96" y="137.16"/>
-<instance part="D4" gate="G$1" x="60.96" y="129.54"/>
-<instance part="D5" gate="G$1" x="60.96" y="121.92"/>
-<instance part="D6" gate="G$1" x="60.96" y="114.3"/>
 <instance part="SUPPLY2" gate="G$1" x="195.58" y="149.86" rot="MR0"/>
 <instance part="GND2" gate="1" x="195.58" y="139.7" rot="MR0"/>
@@
 <instance part="GND3" gate="1" x="96.52" y="43.18"/>
 <instance part="U1" gate="G$1" x="175.26" y="132.08"/>
-<instance part="GND4" gate="1" x="68.58" y="109.22"/>
-<instance part="SUPPLY1" gate="G$1" x="119.38" y="71.12"/>
-<instance part="C1" gate="G$1" x="119.38" y="63.5"/>
-<instance part="C2" gate="G$1" x="129.54" y="63.5"/>
-<instance part="SUPPLY4" gate="G$1" x="129.54" y="71.12"/>
-<instance part="GND1" gate="1" x="119.38" y="53.34"/>
-<instance part="GND5" gate="1" x="129.54" y="53.34"/>
+<instance part="GND4" gate="1" x="68.58" y="132.08"/>
 </instances>
 <busses>
@@
 <net name="KEY4" class="0">
 <segment>
-<wire x1="43.18" y1="129.54" x2="45.72" y2="129.54" width="0.1524" layer="91"/>
-<label x="43.18" y="129.54" size="1.27" layer="95" rot="R180" xref="yes"/>
-<pinref part="SW4" gate="G$1" pin="NO"/>
-</segment>
-<segment>
 <wire x1="157.48" y1="121.92" x2="160.02" y2="121.92" width="0.1524" layer="91"/>
 <label x="157.48" y="121.92" size="1.27" layer="95" rot="R180" xref="yes"/>
@@
 <net name="KEY5" class="0">
 <segment>
-<wire x1="43.18" y1="121.92" x2="45.72" y2="121.92" width="0.1524" layer="91"/>
-<label x="43.18" y="121.92" size="1.27" layer="95" rot="R180" xref="yes"/>
-<pinref part="SW5" gate="G$1" pin="NO"/>
-</segment>
-<segment>
 <wire x1="157.48" y1="119.38" x2="160.02" y2="119.38" width="0.1524" layer="91"/>
 <label x="157.48" y="119.38" size="1.27" layer="95" rot="R180" xref="yes"/>
@@
 </net>
 <net name="KEY6" class="0">
-<segment>
-<wire x1="43.18" y1="114.3" x2="45.72" y2="114.3" width="0.1524" layer="91"/>
-<label x="43.18" y="114.3" size="1.27" layer="95" rot="R180" xref="yes"/>
-<pinref part="SW6" gate="G$1" pin="NO"/>
-</segment>
 <segment>
 <wire x1="157.48" y1="116.84" x2="160.02" y2="116.84" width="0.1524" layer="91"/>
@@
 </segment>
 <segment>
-<wire x1="63.5" y1="114.3" x2="68.58" y2="114.3" width="0.1524" layer="91"/>
 <pinref part="GND4" gate="1" pin="GND"/>
-<wire x1="68.58" y1="114.3" x2="68.58" y2="111.76" width="0.1524" layer="91"/>
-<wire x1="63.5" y1="121.92" x2="68.58" y2="121.92" width="0.1524" layer="91"/>
-<wire x1="68.58" y1="121.92" x2="68.58" y2="114.3" width="0.1524" layer="91"/>
-<junction x="68.58" y="114.3"/>
-<wire x1="68.58" y1="121.92" x2="68.58" y2="129.54" width="0.1524" layer="91"/>
-<junction x="68.58" y="121.92"/>
-<wire x1="68.58" y1="129.54" x2="63.5" y2="129.54" width="0.1524" layer="91"/>
-<wire x1="68.58" y1="129.54" x2="68.58" y2="137.16" width="0.1524" layer="91"/>
-<junction x="68.58" y="129.54"/>
+<wire x1="68.58" y1="137.16" x2="68.58" y2="134.62" width="0.1524" layer="91"/>
 <wire x1="68.58" y1="137.16" x2="63.5" y2="137.16" width="0.1524" layer="91"/>
 <wire x1="68.58" y1="137.16" x2="68.58" y2="144.78" width="0.1524" layer="91"/>
@@
 <pinref part="D2" gate="G$1" pin="C"/>
 <pinref part="D3" gate="G$1" pin="C"/>
-<pinref part="D4" gate="G$1" pin="C"/>
-<pinref part="D5" gate="G$1" pin="C"/>
-<pinref part="D6" gate="G$1" pin="C"/>
-</segment>
-<segment>
-<pinref part="C1" gate="G$1" pin="2"/>
-<pinref part="GND1" gate="1" pin="GND"/>
-<wire x1="119.38" y1="55.88" x2="119.38" y2="58.42" width="0.1524" layer="91"/>
-</segment>
-<segment>
-<pinref part="C2" gate="G$1" pin="2"/>
-<pinref part="GND5" gate="1" pin="GND"/>
-<wire x1="129.54" y1="55.88" x2="129.54" y2="58.42" width="0.1524" layer="91"/>
 </segment>
 </net>
@@
 <pinref part="SUPPLY3" gate="G$1" pin="VCC"/>
 <wire x1="96.52" y1="78.74" x2="96.52" y2="81.28" width="0.1524" layer="91"/>
-</segment>
-<segment>
-<pinref part="SUPPLY1" gate="G$1" pin="VCC"/>
-<pinref part="C1" gate="G$1" pin="1"/>
-<wire x1="119.38" y1="71.12" x2="119.38" y2="68.58" width="0.1524" layer="91"/>
-</segment>
-<segment>
-<pinref part="C2" gate="G$1" pin="1"/>
-<pinref part="SUPPLY4" gate="G$1" pin="VCC"/>
-<wire x1="129.54" y1="71.12" x2="129.54" y2="68.58" width="0.1524" layer="91"/>
 </segment>
 </net>
@@
 </segment>
 </net>
-<net name="N$4" class="0">
-<segment>
-<pinref part="D4" gate="G$1" pin="A"/>
-<pinref part="SW4" gate="G$1" pin="COM"/>
-<wire x1="55.88" y1="129.54" x2="58.42" y2="129.54" width="0.1524" layer="91"/>
-</segment>
-</net>
-<net name="N$5" class="0">
-<segment>
-<pinref part="D5" gate="G$1" pin="A"/>
-<pinref part="SW5" gate="G$1" pin="COM"/>
-<wire x1="55.88" y1="121.92" x2="58.42" y2="121.92" width="0.1524" layer="91"/>
-</segment>
-</net>
-<net name="N$6" class="0">
-<segment>
-<pinref part="D6" gate="G$1" pin="A"/>
-<pinref part="SW6" gate="G$1" pin="COM"/>
-<wire x1="55.88" y1="114.3" x2="58.42" y2="114.3" width="0.1524" layer="91"/>
-</segment>
-</net>
